File: ice40-breakout-pcb.kicad_pcb (KiCad board)
At the start: 2 copper layers, 56 x 71.8 mm, 63 parts, among them J1 USB_B_Micro, J2 USB_Break_Out, J3 Conn_02x16_Odd_Even, J4 Conn_02x16_Odd_Even, J5 Conn_02x16_Odd_Even, J6 Conn_02x04_Odd_Even, U1 SIT2001BI-S2-33E-12.000000G, U2 TLV73333PDBV, U3 TLV73312PDBV, U4 AT25SF081-SHD-X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

Commit message: Label main external connectors.
Other:
- board text added: "1"
- board text added: "10"
- board text added: "11"
- board text added: "12"
- board text added: "13"
- board text added: "14"
- board text added: "15"
- board text added: "16"
- board text added: "17"
- board text added: "18"
- board text added: "19"
- board text added: "2"
- board text added: "20"
- board text added: "21"
- board text added: "22"
- board text added: "23"
- board text added: "24"
- board text added: "25"
- board text added: "26"
- board text added: "27"
- board text added: "28"
- board text added: "29"
- board text added: "3"
- board text added: "30"
- board text added: "31"
- board text added: "32"
- board text added: "33"
- board text added: "34"
- board text added: "35"
- board text added: "36"
- board text added: "4"
- board text added: "5"
- board text added: "6"
- board text added: "7"
- board text added: "8"
- board text added: "9"
Changed lines of the file:
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@@
   (general
     (thickness 1.6)
-    (drawings 12)
+    (drawings 60)
     (tracks 849)
     (zones 0)
@@
     (descr "Through hole straight pin header, 2x05, 2.54mm pitch, double rows")
     (tags "Through hole pin header THT 2x05 2.54mm double row")
-    (fp_text reference J6 (at 1.25 12.5) (layer F.SilkS)
+    (fp_text reference J6 (at 1.25 12.5) (layer F.SilkS) hide
       (effects (font (size 0.8 0.8) (thickness 0.15)))
     )
@@
     (descr "Through hole straight pin header, 2x16, 2.54mm pitch, double rows")
     (tags "Through hole pin header THT 2x16 2.54mm double row")
-    (fp_text reference J5 (at 1.27 -2.4 90) (layer F.SilkS)
+    (fp_text reference J5 (at 1.27 -2.4 90) (layer F.SilkS) hide
       (effects (font (size 0.8 0.8) (thickness 0.15)))
     )
@@
     (descr "Through hole straight pin header, 2x16, 2.54mm pitch, double rows")
     (tags "Through hole pin header THT 2x16 2.54mm double row")
-    (fp_text reference J4 (at 1.27 -2.4) (layer F.SilkS)
+    (fp_text reference J4 (at 1.27 -2.4) (layer F.SilkS) hide
       (effects (font (size 0.8 0.8) (thickness 0.15)))
     )
@@
     (descr "Through hole straight pin header, 2x16, 2.54mm pitch, double rows")
     (tags "Through hole pin header THT 2x16 2.54mm double row")
-    (fp_text reference J3 (at 1.25 -2.3) (layer F.SilkS)
+    (fp_text reference J3 (at 1.25 -2.3) (layer F.SilkS) hide
       (effects (font (size 0.8 0.8) (thickness 0.15)))
     )
@@
     )
   )
+  (gr_text 36 (at 140.425 104.7 90) (layer F.SilkS)
+    (effects (font (size 0.8 0.8) (thickness 0.153)))
+  )
+  (gr_text 35 (at 140.425 102.15 90) (layer F.SilkS)
+    (effects (font (size 0.8 0.8) (thickness 0.153)))
+  )
+  (gr_text 34 (at 140.425 99.625 90) (layer F.SilkS)
+    (effects (font (size 0.8 0.8) (thickness 0.153)))
+  )
+  (gr_text 33 (at 140.425 97.075 90) (layer F.SilkS)
+    (effects (font (size 0.8 0.8) (thickness 0.153)))
+  )
+  (gr_text 3V3 (at 140.425 94.55 90) (layer F.SilkS)
+    (effects (font (size 0.8 0.8) (thickness 0.153)))
+  )
+  (gr_text GND (at 140.425 92 90) (layer F.SilkS)
+    (effects (font (size 0.8 0.8) (thickness 0.153)))
+  )
+  (gr_text 32 (at 140.425 89.475 90) (layer F.SilkS)
+    (effects (font (size 0.8 0.8) (thickness 0.153)))
+  )
+  (gr_text 31 (at 140.425 86.925 90) (layer F.SilkS)
+    (effects (font (size 0.8 0.8) (thickness 0.153)))
+  )
+  (gr_text 30 (at 140.425 84.375 90) (layer F.SilkS)
+    (effects (font (size 0.8 0.8) (thickness 0.153)))
+  )
+  (gr_text 29 (at 140.425 81.85 90) (layer F.SilkS)
+    (effects (font (size 0.8 0.8) (thickness 0.153)))
+  )
+  (gr_text 3V3 (at 140.425 79.3 90) (layer F.SilkS)
+    (effects (font (size 0.8 0.8) (thickness 0.153)))
+  )
+  (gr_text GND (at 140.425 76.775 90) (layer F.SilkS)
+    (effects (font (size 0.8 0.8) (thickness 0.153)))
+  )
+  (gr_text 28 (at 140.425 74.225 90) (layer F.SilkS)
+    (effects (font (size 0.8 0.8) (thickness 0.153)))
+  )
+  (gr_text 27 (at 140.425 71.675 90) (layer F.SilkS)
+    (effects (font (size 0.8 0.8) (thickness 0.153)))
+  )
+  (gr_text 26 (at 140.425 69.15 90) (layer F.SilkS)
+    (effects (font (size 0.8 0.8) (thickness 0.153)))
+  )
+  (gr_text 25 (at 140.425 66.6 90) (layer F.SilkS)
+    (effects (font (size 0.8 0.8) (thickness 0.153)))
+  )
+  (gr_text 24 (at 139.05 65.325) (layer F.SilkS)
+    (effects (font (size 0.8 0.8) (thickness 0.153)))
+  )
+  (gr_text 23 (at 136.5 65.3) (layer F.SilkS)
+    (effects (font (size 0.8 0.8) (thickness 0.153)))
+  )
+  (gr_text 22 (at 133.975 65.3) (layer F.SilkS)
+    (effects (font (size 0.8 0.8) (thickness 0.153)))
+  )
+  (gr_text 21 (at 131.425 65.3) (layer F.SilkS)
+    (effects (font (size 0.8 0.8) (thickness 0.153)))
+  )
+  (gr_text 3V3 (at 128.9 65.3) (layer F.SilkS)
+    (effects (font (size 0.8 0.8) (thickness 0.153)))
+  )
+  (gr_text GND (at 126.35 65.3) (layer F.SilkS)
+    (effects (font (size 0.8 0.8) (thickness 0.153)))
+  )
+  (gr_text 20 (at 123.825 65.3) (layer F.SilkS)
+    (effects (font (size 0.8 0.8) (thickness 0.153)))
+  )
+  (gr_text 19 (at 121.275 65.3) (layer F.SilkS)
+    (effects (font (size 0.8 0.8) (thickness 0.153)))
+  )
+  (gr_text 18 (at 118.725 65.3) (layer F.SilkS)
+    (effects (font (size 0.8 0.8) (thickness 0.153)))
+  )
+  (gr_text 17 (at 116.2 65.3) (layer F.SilkS)
+    (effects (font (size 0.8 0.8) (thickness 0.153)))
+  )
+  (gr_text 3V3 (at 113.65 65.3) (layer F.SilkS)
+    (effects (font (size 0.8 0.8) (thickness 0.153)))
+  )
+  (gr_text GND (at 111.125 65.3) (layer F.SilkS)
+    (effects (font (size 0.8 0.8) (thickness 0.153)))
+  )
+  (gr_text 16 (at 108.575 65.3) (layer F.SilkS)
+    (effects (font (size 0.8 0.8) (thickness 0.153)))
+  )
+  (gr_text 15 (at 106.025 65.3) (layer F.SilkS)
+    (effects (font (size 0.8 0.8) (thickness 0.153)))
+  )
+  (gr_text 14 (at 103.5 65.35) (layer F.SilkS)
+    (effects (font (size 0.8 0.8) (thickness 0.153)))
+  )
+  (gr_text 3V3 (at 99.65 76.75 90) (layer F.SilkS)
+    (effects (font (size 0.8 0.8) (thickness 0.153)))
+  )
+  (gr_text GND (at 99.65 79.3 90) (layer F.SilkS)
+    (effects (font (size 0.8 0.8) (thickness 0.153)))
+  )
+  (gr_text 3V3 (at 99.65 92 90) (layer F.SilkS)
+    (effects (font (size 0.8 0.8) (thickness 0.153)))
+  )
+  (gr_text GND (at 99.65 94.525 90) (layer F.SilkS)
+    (effects (font (size 0.8 0.8) (thickness 0.153)))
+  )
+  (gr_text 1 (at 99.65 104.7 90) (layer F.SilkS)
+    (effects (font (size 0.8 0.8) (thickness 0.153)))
+  )
+  (gr_text 2 (at 99.65 102.15 90) (layer F.SilkS)
+    (effects (font (size 0.8 0.8) (thickness 0.153)))
+  )
+  (gr_text 3 (at 99.65 99.625 90) (layer F.SilkS)
+    (effects (font (size 0.8 0.8) (thickness 0.153)))
+  )
+  (gr_text 4 (at 99.675 97.075 90) (layer F.SilkS)
+    (effects (font (size 0.8 0.8) (thickness 0.153)))
+  )
+  (gr_text 5 (at 99.65 89.45 90) (layer F.SilkS)
+    (effects (font (size 0.8 0.8) (thickness 0.153)))
+  )
+  (gr_text 6 (at 99.65 86.925 90) (layer F.SilkS)
+    (effects (font (size 0.8 0.8) (thickness 0.153)))
+  )
+  (gr_text 7 (at 99.65 84.375 90) (layer F.SilkS)
+    (effects (font (size 0.8 0.8) (thickness 0.153)))
+  )
+  (gr_text 8 (at 99.65 81.85 90) (layer F.SilkS)
+    (effects (font (size 0.8 0.8) (thickness 0.153)))
+  )
+  (gr_text 9 (at 99.65 74.225 90) (layer F.SilkS)
+    (effects (font (size 0.8 0.8) (thickness 0.153)))
+  )
+  (gr_text 10 (at 99.65 71.675 90) (layer F.SilkS)
+    (effects (font (size 0.8 0.8) (thickness 0.153)))
+  )
+  (gr_text 11 (at 99.65 69.125 90) (layer F.SilkS)
+    (effects (font (size 0.8 0.8) (thickness 0.153)))
+  )
+  (gr_text 13 (at 100.95 65.3) (layer F.SilkS)
+    (effects (font (size 0.8 0.8) (thickness 0.153)))
+  )
+  (gr_text 12 (at 99.65 66.6 90) (layer F.SilkS)
+    (effects (font (size 0.8 0.8) (thickness 0.153)))
+  )
   (gr_text 3V3 (at 106.45 108.45) (layer F.SilkS)
